Commit message: Updating the joint state publisher

File: biometra_description/urdf/thermocycler.urdf.xacro (robot description, xacro)
@@ -1,11 +1,11 @@
 <?xml version="1.0"?>
-<robot name="Thermocycler" xmlns:xacro="http://www.ros.org/wiki/xacro">
+<robot name="Biometra" xmlns:xacro="http://www.ros.org/wiki/xacro">
   <!-- Links -->
-  <xacro:macro name="Thermocycler" params = "prefix">
-  <link name="${prefix}thermocycler_base">
+  <xacro:macro name="Biometra" params = "prefix">
+  <link name="${prefix}biometra_base">
     <visual>
       <origin xyz="0 0.5 1.042" rpy="1.5708 0 0"/>
       <geometry>
-        <mesh filename="package://pf400_description/meshes/thermocycler_base.STL" scale="0.001 0.001 0.001"/>
+        <mesh filename="package://pf400_description/meshes/biometra_base.STL" scale="0.001 0.001 0.001"/>
       </geometry>
       <material name="light_grey"/>
@@ -13,14 +13,14 @@
     <collision>
       <geometry>
-        <mesh filename="package://pf400_description/meshes/thermocycler_base.STL" scale="0.001 0.001 0.001"/>
+        <mesh filename="package://pf400_description/meshes/biometra_base.STL" scale="0.001 0.001 0.001"/>
       </geometry>
       <origin xyz="0 0.5 1.042" rpy="1.5708 0 0"/>
     </collision>
   </link>
-  <link name="${prefix}thermocycler_cap">
+  <link name="${prefix}biometra_cap">
     <visual>
       <origin xyz="0 0 0" rpy="0 0 0"/>
       <geometry>
-        <mesh filename="package://pf400_description/meshes/thermocycler_cap.STL" scale="0.001 0.001 0.001"/>
+        <mesh filename="package://pf400_description/meshes/biometra_cap.STL" scale="0.001 0.001 0.001"/>
       </geometry>
       <material name="red"/>
@@ -28,14 +28,14 @@
     <collision>
       <geometry>
-        <mesh filename="package://pf400_description/meshes/thermocycler_cap.STL" scale="0.001 0.001 0.001"/>
+        <mesh filename="package://pf400_description/meshes/biometra_cap.STL" scale="0.001 0.001 0.001"/>
       </geometry>
       <origin xyz="0 0 0" rpy="0 0 0"/>
     </collision>
   </link>
-  <link name="${prefix}thermocycler_base2">
+  <link name="${prefix}biometra_base2">
     <visual>
       <origin xyz="0 0.5 1.042" rpy="1.5708 0 0"/>
       <geometry>
-        <mesh filename="package://pf400_description/meshes/thermocycler_base.STL" scale="0.001 0.001 0.001"/>
+        <mesh filename="package://pf400_description/meshes/biometra_base.STL" scale="0.001 0.001 0.001"/>
       </geometry>
       <material name="light_grey"/>
@@ -43,14 +43,14 @@
     <collision>
       <geometry>
-        <mesh filename="package://pf400_description/meshes/thermocycler_base.STL" scale="0.001 0.001 0.001"/>
+        <mesh filename="package://pf400_description/meshes/biometra_base.STL" scale="0.001 0.001 0.001"/>
       </geometry>
       <origin xyz="0 0.5 1.042" rpy="1.5708 0 0"/>
     </collision>
   </link>
-  <link name="${prefix}thermocycler_cap2">
+  <link name="${prefix}biometra_cap2">
     <visual>
       <origin xyz="0 0 0" rpy="0 0 0"/>
       <geometry>
-        <mesh filename="package://pf400_description/meshes/thermocycler_cap.STL" scale="0.001 0.001 0.001"/>
+        <mesh filename="package://pf400_description/meshes/biometra_cap.STL" scale="0.001 0.001 0.001"/>
       </geometry>
       <material name="red"/>
@@ -58,5 +58,5 @@
     <collision>
       <geometry>
-        <mesh filename="package://pf400_description/meshes/thermocycler_cap.STL" scale="0.001 0.001 0.001"/>
+        <mesh filename="package://pf400_description/meshes/biometra_cap.STL" scale="0.001 0.001 0.001"/>
       </geometry>
       <origin xyz="0 0 0" rpy="0 0 0"/>
@@ -64,17 +64,17 @@
   </link>
   <!-- Joints -->
-  <joint name="Thermocycler_Cap" type="fixed">
-    <parent link="${prefix}thermocycler_base"/>
-    <child link="${prefix}thermocycler_cap"/>
+  <joint name="Biometra_Cap" type="fixed">
+    <parent link="${prefix}biometra_base"/>
+    <child link="${prefix}biometra_cap"/>
     <axis xyz="-1 0 0"/>
     <origin xyz="0 0.466 1.05" rpy="0.4 0 0"/>
     <limit effort="1000.0" lower="1.2" upper="1.2" velocity="0.5"/>
   </joint>
-  <joint name="Thermocycler_Cap2" type="fixed">
-    <parent link="${prefix}thermocycler_base2"/>
-    <child link="${prefix}thermocycler_cap2"/>
+  <joint name="Biometra_Cap2" type="revolute">
+    <parent link="${prefix}biometra_base2"/>
+    <child link="${prefix}biometra_cap2"/>
     <axis xyz="-1 0 0"/>
     <origin xyz="0 0.466 1.05" rpy="1.5708 0 0"/>
-    <limit effort="1000.0" lower="1.2" upper="1.2" velocity="0.5"/>
+    <limit effort="1000.0" lower="0" upper="1.2" velocity="0.5"/>
   </joint>
   </xacro:macro>
