Commit message: Clean up

File: biometra_description/urdf/biometra.urdf.xacro (robot description, xacro)
@@ -7,5 +7,5 @@
       <origin xyz="0 0.5 1.042" rpy="1.5708 0 0"/>
       <geometry>
-        <mesh filename="package://pf400_description/meshes/biometra_base.STL" scale="0.001 0.001 0.001"/>
+        <mesh filename="package://biometra_description/meshes/biometra_base.STL" scale="0.001 0.001 0.001"/>
       </geometry>
       <material name="light_grey"/>
@@ -13,5 +13,5 @@
     <collision>
       <geometry>
-        <mesh filename="package://pf400_description/meshes/biometra_base.STL" scale="0.001 0.001 0.001"/>
+        <mesh filename="package://biometra_description/meshes/biometra_base.STL" scale="0.001 0.001 0.001"/>
       </geometry>
       <origin xyz="0 0.5 1.042" rpy="1.5708 0 0"/>
@@ -22,5 +22,5 @@
       <origin xyz="0 0 0" rpy="0 0 0"/>
       <geometry>
-        <mesh filename="package://pf400_description/meshes/biometra_cap.STL" scale="0.001 0.001 0.001"/>
+        <mesh filename="package://biometra_description/meshes/biometra_cap.STL" scale="0.001 0.001 0.001"/>
       </geometry>
       <material name="red"/>
@@ -28,5 +28,5 @@
     <collision>
       <geometry>
-        <mesh filename="package://pf400_description/meshes/biometra_cap.STL" scale="0.001 0.001 0.001"/>
+        <mesh filename="package://biometra_description/meshes/biometra_cap.STL" scale="0.001 0.001 0.001"/>
       </geometry>
       <origin xyz="0 0 0" rpy="0 0 0"/>
@@ -37,5 +37,5 @@
       <origin xyz="0 0.5 1.042" rpy="1.5708 0 0"/>
       <geometry>
-        <mesh filename="package://pf400_description/meshes/biometra_base.STL" scale="0.001 0.001 0.001"/>
+        <mesh filename="package://biometra_description/meshes/biometra_base.STL" scale="0.001 0.001 0.001"/>
       </geometry>
       <material name="light_grey"/>
@@ -43,5 +43,5 @@
     <collision>
       <geometry>
-        <mesh filename="package://pf400_description/meshes/biometra_base.STL" scale="0.001 0.001 0.001"/>
+        <mesh filename="package://biometra_description/meshes/biometra_base.STL" scale="0.001 0.001 0.001"/>
       </geometry>
       <origin xyz="0 0.5 1.042" rpy="1.5708 0 0"/>
@@ -52,5 +52,5 @@
       <origin xyz="0 0 0" rpy="0 0 0"/>
       <geometry>
-        <mesh filename="package://pf400_description/meshes/biometra_cap.STL" scale="0.001 0.001 0.001"/>
+        <mesh filename="package://biometra_description/meshes/biometra_cap.STL" scale="0.001 0.001 0.001"/>
       </geometry>
       <material name="red"/>
@@ -58,5 +58,5 @@
     <collision>
       <geometry>
-        <mesh filename="package://pf400_description/meshes/biometra_cap.STL" scale="0.001 0.001 0.001"/>
+        <mesh filename="package://biometra_description/meshes/biometra_cap.STL" scale="0.001 0.001 0.001"/>
       </geometry>
       <origin xyz="0 0 0" rpy="0 0 0"/>

Commit message: Changin the joint type

File: biometra_description/urdf/biometra.urdf.xacro (robot description, xacro)
@@ -71,5 +71,5 @@
     <limit effort="1000.0" lower="1.2" upper="1.2" velocity="0.5"/>
   </joint>
-  <joint name="Biometra_Cap2" type="revolute">
+  <joint name="Biometra_Cap2" type="prismatic">
     <parent link="${prefix}biometra_base2"/>
     <child link="${prefix}biometra_cap2"/>

Commit message: Clean up

File: biometra_description/urdf/biometra.urdf.xacro (robot description, xacro)
@@ -64,17 +64,17 @@
   </link>
   <!-- Joints -->
-  <joint name="Biometra_Cap" type="fixed">
+  <joint name="Biometra_Cap" type="revolute">
     <parent link="${prefix}biometra_base"/>
     <child link="${prefix}biometra_cap"/>
     <axis xyz="-1 0 0"/>
-    <origin xyz="0 0.466 1.05" rpy="0.4 0 0"/>
-    <limit effort="1000.0" lower="1.2" upper="1.2" velocity="0.5"/>
+    <origin xyz="0 0.466 1.05" rpy="1.5708 0 0"/>
+    <limit effort="1000.0" lower="0.0" upper="1.2" velocity="0.5"/>
   </joint>
-  <joint name="Biometra_Cap2" type="prismatic">
+  <joint name="Biometra_Cap2" type="revolute">
     <parent link="${prefix}biometra_base2"/>
     <child link="${prefix}biometra_cap2"/>
     <axis xyz="-1 0 0"/>
     <origin xyz="0 0.466 1.05" rpy="1.5708 0 0"/>
-    <limit effort="1000.0" lower="0" upper="1.2" velocity="0.5"/>
+    <limit effort="1000.0" lower="0.0" upper="1.2" velocity="0.5"/>
   </joint>
   </xacro:macro>
