Commit message: Updating the new module cart mesh

File: biometra_description/urdf/module_carts.urdf.xacro (robot description, xacro)
@@ -3,9 +3,9 @@
   <!-- Links -->
   <xacro:macro name="Module_Carts" params = "prefix">
-  <link name="${prefix}cart_1">
+  <link name="${prefix}cart_2">
     <visual>
       <origin xyz="0 0 0" rpy="0 0 0"/>
       <geometry>
-        <mesh filename="package://pf400_description/meshes/module_cart.stl" scale="1 1 1"/>
+        <mesh filename="package://biometra_description/meshes/module_cart.stl" scale="1 1 1"/>
       </geometry>
       <material name="darkbluegreen"/>
@@ -13,186 +13,9 @@
     <collision>
       <geometry>
-        <mesh filename="package://pf400_description/meshes/module_cart.stl" scale="1 1 1"/>
+        <mesh filename="package://biometra_description/meshes/module_cart.stl" scale="1 1 1"/>
       </geometry>
       <origin xyz="0 0 0" rpy="0 0 0"/>
     </collision>
   </link>
-  <link name="${prefix}cart_2">
-    <visual>
-      <origin xyz="0 0 0" rpy="0 0 0"/>
-      <geometry>
-        <mesh filename="package://pf400_description/meshes/module_cart.stl" scale="1 1 1"/>
-      </geometry>
-      <material name="darkbluegreen"/>
-    </visual>
-    <collision>
-      <geometry>
-        <mesh filename="package://pf400_description/meshes/module_cart.stl" scale="1 1 1"/>
-      </geometry>
-      <origin xyz="0 0 0" rpy="0 0 0"/>
-    </collision>
-  </link>
-  <link name="${prefix}cart_3">
-    <visual>
-      <origin xyz="0 0 0" rpy="0 0 0"/>
-      <geometry>
-        <mesh filename="package://pf400_description/meshes/module_cart.stl" scale="1 1 1"/>
-      </geometry>
-      <material name="darkbluegreen"/>
-    </visual>
-    <collision>
-      <geometry>
-        <mesh filename="package://pf400_description/meshes/module_cart.stl" scale="1 1 1"/>
-      </geometry>
-      <origin xyz="0 0 0" rpy="0 0 0"/>
-    </collision>
-  </link>
-  <link name="${prefix}cart_4">
-    <visual>
-      <origin xyz="0 0 0" rpy="0 0 0"/>
-      <geometry>
-        <mesh filename="package://pf400_description/meshes/module_cart.stl" scale="1 1 1"/>
-      </geometry>
-      <material name="darkbluegreen"/>
-    </visual>
-    <collision>
-      <geometry>
-        <mesh filename="package://pf400_description/meshes/module_cart.stl" scale="1 1 1"/>
-      </geometry>
-      <origin xyz="0 0 0" rpy="0 0 0"/>
-    </collision>
-  </link>
-  <link name="${prefix}cart_5">
-    <visual>
-      <origin xyz="0 0 0" rpy="0 0 0"/>
-      <geometry>
-        <mesh filename="package://pf400_description/meshes/module_cart.stl" scale="1 1 1"/>
-      </geometry>
-      <material name="darkbluegreen"/>
-    </visual>
-    <collision>
-      <geometry>
-        <mesh filename="package://pf400_description/meshes/module_cart.stl" scale="1 1 1"/>
-      </geometry>
-      <origin xyz="0 0 0" rpy="0 0 0"/>
-    </collision>
-  </link>
-  <link name="${prefix}cart_6">
-    <visual>
-      <origin xyz="0 0 0" rpy="0 0 0"/>
-      <geometry>
-        <mesh filename="package://pf400_description/meshes/module_cart.stl" scale="1 1 1"/>
-      </geometry>
-      <material name="darkbluegreen"/>
-    </visual>
-    <collision>
-      <geometry>
-        <mesh filename="package://pf400_description/meshes/module_cart.stl" scale="1 1 1"/>
-      </geometry>
-      <origin xyz="0 0 0" rpy="0 0 0"/>
-    </collision>
-  </link>
-  <link name="${prefix}cart_7">
-    <visual>
-      <origin xyz="0 0 0" rpy="0 0 0"/>
-      <geometry>
-        <mesh filename="package://pf400_description/meshes/module_cart.stl" scale="1 1 1"/>
-      </geometry>
-      <material name="darkbluegreen"/>
-    </visual>
-    <collision>
-      <geometry>
-        <mesh filename="package://pf400_description/meshes/module_cart.stl" scale="1 1 1"/>
-      </geometry>
-      <origin xyz="0 0 0" rpy="0 0 0"/>
-    </collision>
-  </link>
-  <link name="${prefix}cart_8">
-    <visual>
-      <origin xyz="0 0 0" rpy="0 0 0"/>
-      <geometry>
-        <mesh filename="package://pf400_description/meshes/module_cart.stl" scale="1 1 1"/>
-      </geometry>
-      <material name="darkbluegreen"/>
-    </visual>
-    <collision>
-      <geometry>
-        <mesh filename="package://pf400_description/meshes/module_cart.stl" scale="1 1 1"/>
-      </geometry>
-      <origin xyz="0 0 0" rpy="0 0 0"/>
-    </collision>
-  </link>
-  <link name="${prefix}pf400_cart">
-    <visual>
-      <origin xyz="-1.592 0.2605 -0.015" rpy="1.5708 0 0"/>
-      <geometry>
-        <mesh filename="package://pf400_description/meshes/pf400_table.STL" scale="0.001 0.001 0.001"/>
-      </geometry>
-      <material name="darkbluegreen"/>
-    </visual>
-    <collision>
-      <geometry>
-        <mesh filename="package://pf400_description/meshes/pf400_table.STL" scale="0.001 0.001 0.001"/>
-      </geometry>
-      <origin xyz="-1.592 0.261 -0.015" rpy="1.5708 0 0"/>
-    </collision>
-  </link>
-  <!-- Joints -->
-  <joint name="pf400_cart_to_cart_1" type="fixed">
-    <parent link="${prefix}pf400_cart"/>
-    <child link="${prefix}cart_1"/>
-    <axis xyz="0 0 1"/>
-    <origin xyz="1.0 0.83 0" rpy="0 0 0"/>
-    <limit effort="1000.0" lower="0" upper="0" velocity="0.5"/>
-  </joint>
-  <joint name="pf400_cart_to_cart_2" type="fixed">
-    <parent link="${prefix}pf400_cart"/>
-    <child link="${prefix}cart_2"/>
-    <axis xyz="0 0 1"/>
-    <origin xyz="0.25 0.83 0" rpy="0 0 0"/>
-    <limit effort="1000.0" lower="0" upper="0" velocity="0.5"/>
-  </joint>
-  <joint name="pf400_cart_to_cart_3" type="fixed">
-    <parent link="${prefix}pf400_cart"/>
-    <child link="${prefix}cart_3"/>
-    <axis xyz="0 0 1"/>
-    <origin xyz="-0.50 0.83  0" rpy="0 0 0"/>
-    <limit effort="1000.0" lower="0" upper="0" velocity="0.5"/>
-  </joint>
-  <joint name="pf400_cart_to_cart_4" type="fixed">
-    <parent link="${prefix}pf400_cart"/>
-    <child link="${prefix}cart_4"/>
-    <axis xyz="0 0 1"/>
-    <origin xyz="-1.25 0.83  0" rpy="0 0 0"/>
-    <limit effort="1000.0" lower="0" upper="0" velocity="0.5"/>
-  </joint>
-  <joint name="pf400_cart_to_cart_5" type="fixed">
-    <parent link="${prefix}pf400_cart"/>
-    <child link="${prefix}cart_5"/>
-    <axis xyz="0 0 1"/>
-    <origin xyz="1.00 -0.46 0" rpy="0 0 0"/>
-    <limit effort="1000.0" lower="0" upper="0" velocity="0.5"/>
-  </joint>
-  <joint name="pf400_cart_to_cart_6" type="fixed">
-    <parent link="${prefix}pf400_cart"/>
-    <child link="${prefix}cart_6"/>
-    <axis xyz="0 0 1"/>
-    <origin xyz="0.25 -0.46 0" rpy="0 0 0"/>
-    <limit effort="1000.0" lower="0" upper="0" velocity="0.5"/>
-  </joint>
-  <joint name="pf400_cart_to_cart_7" type="fixed">
-    <parent link="${prefix}pf400_cart"/>
-    <child link="${prefix}cart_7"/>
-    <axis xyz="0 0 1"/>
-    <origin xyz="-0.50 -0.46 0" rpy="0 0 0"/>
-    <limit effort="1000.0" lower="0" upper="0" velocity="0.5"/>
-  </joint>
-  <joint name="pf400_cart_to_cart_8" type="fixed">
-    <parent link="${prefix}pf400_cart"/>
-    <child link="${prefix}cart_8"/>
-    <axis xyz="0 0 1"/>
-    <origin xyz="-1.25 -0.46 0" rpy="0 0 0"/>
-    <limit effort="1000.0" lower="0" upper="0" velocity="0.5"/>
-  </joint>
   </xacro:macro>
 </robot>
